File: NeatoLidarInterface.kicad_pcb (KiCad board)
At the start: 2 copper layers, 49 x 69 mm, 8 parts, among them J1 Conn_01x02, J2 Conn_01x04, J3 Conn_01x02, J4 Conn_01x02_Male, J5 Conn_01x02_Male, Q1 PN2222A, U1 STM32BluePill

Commit message: improve JST footprint, add copper fill
Parts:
- J1, J3: footprint Connector_JST:JST_JWPF_B02B-JWPF-SK-R_1x02_P2.00mm_Vertical -> Connector_JST:JST_PH_B2B-PH-K_1x02_P2.00mm_Vertical
- J2: footprint Connector_JST:JST_JWPF_B04B-JWPF-SK-R_1x04_P2.00mm_Vertical -> Connector_JST:JST_PH_B4B-PH-K_1x04_P2.00mm_Vertical
- moved J2 0.29 mm to (185.9, 21.1), turned to 270 degrees
- moved J3 0.28 mm to (185.9, 35.3), turned to 270 degrees
- moved J1 0.28 mm to (185.9, 9.91), turned to 270 degrees
Routing:
- net Net-(J1-Pad2): track 40.3 -> 39.5 mm
- added copper zone on B.Cu, net GND
- added copper zone on F.Cu, net GND
Other:
- board text added: "1K"
- board text added: "2N2222"
- board text added: "B"
- board text added: "C"
- board text added: "E"
- board text added: "Ext. 5V"
- board text added: "USB this end"
- board text removed: "Ext 5V"
