File: NeatoLidarInterface.sch (KiCad schematic (older format))
At the start: 8 parts, among them J1 Conn_01x02, J2 Conn_01x04, J3 Conn_01x02, J4 Conn_01x02_Male, J5 Conn_01x02_Male, Q1 PN2222A, U1 STM32BluePill

Commit message: improve JST footprint, add copper fill
Parts:
- J1, J3: footprint Connector_JST:JST_JWPF_B02B-JWPF-SK-R_1x02_P2.00mm_Vertical -> Connector_JST:JST_PH_B2B-PH-K_1x02_P2.00mm_Vertical
- J2: footprint Connector_JST:JST_JWPF_B04B-JWPF-SK-R_1x04_P2.00mm_Vertical -> Connector_JST:JST_PH_B4B-PH-K_1x04_P2.00mm_Vertical
Changed lines of the file:
@@
 F 0 "J3" H 4618 4075 50  0000 C CNN
 F 1 "Conn_01x02" H 4618 4166 50  0000 C CNN
-F 2 "Connector_JST:JST_JWPF_B02B-JWPF-SK-R_1x02_P2.00mm_Vertical" H 4700 4400 50  0001 C CNN
+F 2 "Connector_JST:JST_PH_B2B-PH-K_1x02_P2.00mm_Vertical" H 4700 4400 50  0001 C CNN
 F 3 "~" H 4700 4400 50  0001 C CNN
 	1    4700 4400
@@
 F 0 "J2" H 4650 3350 50  0000 L CNN
 F 1 "Conn_01x04" H 4650 3450 50  0000 L CNN
-F 2 "Connector_JST:JST_JWPF_B04B-JWPF-SK-R_1x04_P2.00mm_Vertical" H 4700 3100 50  0001 C CNN
+F 2 "Connector_JST:JST_PH_B4B-PH-K_1x04_P2.00mm_Vertical" H 4700 3100 50  0001 C CNN
 F 3 "~" H 4700 3100 50  0001 C CNN
 	1    4700 3100
@@
 F 0 "J1" H 4618 1625 50  0000 C CNN
 F 1 "Conn_01x02" H 4618 1716 50  0000 C CNN
-F 2 "Connector_JST:JST_JWPF_B02B-JWPF-SK-R_1x02_P2.00mm_Vertical" H 4700 1950 50  0001 C CNN
+F 2 "Connector_JST:JST_PH_B2B-PH-K_1x02_P2.00mm_Vertical" H 4700 1950 50  0001 C CNN
 F 3 "~" H 4700 1950 50  0001 C CNN
 	1    4700 1950
